Commit message: Changed file structure, added laser max range modifier

File: src/ursa/urdf/robot_description.urdf (robot description, URDF)
Before this commit: robot handheld_hokuyo, 4 links, 3 joints
Links:
- removed link vertical_laser_link
- added link fcu; visual cylinder length=0.05 radius=0.03
- added link hokuyo_link; visual cylinder length=0.05 radius=0.03
- added link lidar_link; visual cylinder length=0.05 radius=0.03
Joints:
- removed joint vertical_laser_link_joint
- added joint fcu: type fixed, parent base_link, child fcu, origin xyz=0 0 0
- added joint hokuyo_link_joint: type fixed, parent base_link, child hokuyo_link, origin xyz=0 0 0.1
- added joint lidar_link_joint: type fixed, parent base_link, child lidar_link, origin xyz=-0.12 0 0 rpy=0 3.1415 0
